Commit message: Update compass_gait_limit_cycle.urdf

File: underactuated/models/compass_gait_limit_cycle.urdf (robot description, URDF)
Before this commit: robot compass_gait, 6 links, 6 joints
Links:
- link ground: geometry visual box size=10 1 -.5

Commit message: Update compass_gait_limit_cycle.urdf

File: underactuated/models/compass_gait_limit_cycle.urdf (robot description, URDF)
Before this commit: robot compass_gait, 6 links, 6 joints
Links:
- link ground: geometry visual box size=10 1 0.1

Commit message: Update compass_gait_limit_cycle.urdf

File: underactuated/models/compass_gait_limit_cycle.urdf (robot description, URDF)
Before this commit: robot compass_gait, 6 links, 6 joints
Links:
- link ground: geometry visual box size=10 1 0.5

Commit message: decreased slope angle

File: underactuated/models/compass_gait_limit_cycle.urdf (robot description, URDF)
Before this commit: robot compass_gait, 6 links, 6 joints
Joints:
- joint ground_is_world: origin xyz=0 0 0 rpy=0 .04 0 -> xyz=0 0 0 rpy=0 .01 0

Commit message: update slope again

File: underactuated/models/compass_gait_limit_cycle.urdf (robot description, URDF)
Before this commit: robot compass_gait, 6 links, 6 joints
Joints:
- joint ground_is_world: origin xyz=0 0 0 rpy=0 .01 0 -> xyz=0 0 0 rpy=0 .03 0
